File: vcf3/vcf3.sch (EAGLE design)
At the start: 99 parts, among them IC1 OPA4130P, IC2 OPA4130P, IC3 OPA134P, Q1 2N3904, Q10 2N3904, Q11 2N3904, Q12 2N3904, Q2 2N3904, Q3 2N3904, Q4 2N3904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

Commit message: fixed the header position in vcf3 and fixed the 2 pole polarity
Connections:
- net N$3: now also IC2A.+IN; no longer IC2B.+IN
- net N$6: now also IC2B.+IN; no longer IC2A.+IN
Changed lines of the file:
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@@
 <pinref part="C2" gate="G$1" pin="1"/>
 <wire x1="40.64" y1="91.44" x2="38.1" y2="91.44" width="0.1524" layer="91"/>
-<wire x1="38.1" y1="91.44" x2="38.1" y2="96.52" width="0.1524" layer="91"/>
 <junction x="38.1" y="91.44"/>
-<wire x1="38.1" y1="96.52" x2="38.1" y2="119.38" width="0.1524" layer="91"/>
-<wire x1="68.58" y1="96.52" x2="38.1" y2="96.52" width="0.1524" layer="91"/>
-<junction x="38.1" y="96.52"/>
-<pinref part="IC2" gate="B" pin="+IN"/>
+<wire x1="38.1" y1="91.44" x2="38.1" y2="116.84" width="0.1524" layer="91"/>
 <pinref part="Q1" gate="G1" pin="C"/>
 <pinref part="Q4" gate="G1" pin="E"/>
+<pinref part="IC2" gate="A" pin="+IN"/>
+<wire x1="38.1" y1="116.84" x2="38.1" y2="119.38" width="0.1524" layer="91"/>
+<wire x1="68.58" y1="116.84" x2="38.1" y2="116.84" width="0.1524" layer="91"/>
+<junction x="38.1" y="116.84"/>
 </segment>
 </net>
@@
 <pinref part="C2" gate="G$1" pin="2"/>
 <wire x1="48.26" y1="91.44" x2="50.8" y2="91.44" width="0.1524" layer="91"/>
-<wire x1="50.8" y1="91.44" x2="50.8" y2="116.84" width="0.1524" layer="91"/>
+<wire x1="50.8" y1="91.44" x2="50.8" y2="96.52" width="0.1524" layer="91"/>
 <junction x="50.8" y="91.44"/>
-<wire x1="50.8" y1="116.84" x2="50.8" y2="119.38" width="0.1524" layer="91"/>
-<wire x1="68.58" y1="116.84" x2="50.8" y2="116.84" width="0.1524" layer="91"/>
-<junction x="50.8" y="116.84"/>
-<pinref part="IC2" gate="A" pin="+IN"/>
 <pinref part="Q2" gate="G1" pin="C"/>
 <pinref part="Q3" gate="G1" pin="E"/>
+<pinref part="IC2" gate="B" pin="+IN"/>
+<wire x1="50.8" y1="96.52" x2="50.8" y2="119.38" width="0.1524" layer="91"/>
+<wire x1="68.58" y1="96.52" x2="50.8" y2="96.52" width="0.1524" layer="91"/>
+<junction x="50.8" y="96.52"/>
 </segment>
 </net>

Commit message: added center freq trimpot to vcf3, fixed v/oct tracking
Parts:
- added CENTER: 20K, dan:TRIM_US-S64W
- R21: value 220k -> 1M
- R47: value 111k -> 91k
- SCALE: value 100K -> 500K
Connections:
- new net N$40: C19.1, CENTER.E, CENTER.S, R47.2, SV5.4, SV6.4
- net +12V: now also CENTER.A; no longer C19.1, R47.2, SV5.4, SV6.4
Other:
- note removed: "trimmer back in here"
- moved on the sheet: C19, SV5, SV6
Changed lines of the file:
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@@
 <part name="FREQ" library="dan" deviceset="US-EVU" device="F2J" value="10K"/>
 <part name="P-7" library="dan" deviceset="-12V" device=""/>
-<part name="P+9" library="dan" deviceset="+12V" device=""/>
 <part name="R44" library="dan" deviceset="R-US_" device="0204/7" value="470k"/>
 <part name="GAIN1" library="dan" deviceset="US-EVU" device="F2J" value="10K"/>
@@
 <part name="R45" library="dan" deviceset="R-US_" device="0207/2V" value="1k"/>
 <part name="R46" library="dan" deviceset="R-US_" device="0207/2V" value="1k"/>
-<part name="R47" library="dan" deviceset="R-US_" device="0204/7" value="111k"/>
+<part name="R47" library="dan" deviceset="R-US_" device="0204/7" value="91k"/>
 <part name="R48" library="dan" deviceset="R-US_" device="0204/7" value="100k"/>
 <part name="R49" library="dan" deviceset="R-US_" device="0207/2V" value="1k"/>
@@
 <part name="MIN1" library="dan" deviceset="PJ301BM" device=""/>
 <part name="GND12" library="dan" deviceset="GND" device=""/>
-<part name="R21" library="dan" deviceset="R-US_" device="0207/2V" value="220k"/>
+<part name="R21" library="dan" deviceset="R-US_" device="0207/2V" value="1M"/>
 <part name="Q9" library="dan" deviceset="2N3904" device=""/>
 <part name="Q10" library="dan" deviceset="2N3904" device=""/>
 <part name="Q11" library="dan" deviceset="2N3904" device=""/>
 <part name="Q12" library="dan" deviceset="2N3904" device=""/>
-<part name="SCALE" library="dan" deviceset="TRIM_US-" device="S64W" value="100K"/>
+<part name="SCALE" library="dan" deviceset="TRIM_US-" device="S64W" value="500K"/>
 <part name="R26" library="dan" deviceset="R-US_" device="0207/2V" value="22k"/>
 <part name="C9" library="dan" deviceset="CPOL-US" device="E2.5-6" value="4.7u"/>
@@
 <part name="IC3" library="dan" deviceset="OPA134" device="P"/>
 <part name="C15" library="dan" deviceset="CPOL-US" device="E2.5-6" value="10u"/>
+<part name="CENTER" library="dan" deviceset="TRIM_US-" device="S64W" value="20K"/>
+<part name="GND14" library="dan" deviceset="GND" device=""/>
 </parts>
 <sheets>
 <sheet>
 <plain>
-<text x="-175.26" y="7.62" size="1.778" layer="91">trimmer back in here</text>
 </plain>
 <instances>
@@
 <instance part="FREQ" gate="G$1" x="-149.86" y="-5.08" rot="MR180"/>
 <instance part="P-7" gate="1" x="-149.86" y="-30.48"/>
-<instance part="P+9" gate="1" x="-149.86" y="20.32"/>
 <instance part="R44" gate="G$1" x="-137.16" y="-5.08"/>
 <instance part="GAIN1" gate="G$1" x="-27.94" y="60.96" rot="MR0"/>
@@
 <instance part="P+5" gate="1" x="-48.26" y="50.8"/>
 <instance part="P-3" gate="1" x="-48.26" y="25.4"/>
-<instance part="C19" gate="G$1" x="-53.34" y="144.78"/>
+<instance part="C19" gate="G$1" x="-187.96" y="12.7"/>
 <instance part="C20" gate="G$1" x="-53.34" y="129.54" rot="R180"/>
 <instance part="P+7" gate="1" x="73.66" y="124.46"/>
@@
 <instance part="SV1" gate="1" x="-152.4" y="76.2"/>
 <instance part="SV2" gate="1" x="-160.02" y="76.2" rot="MR0"/>
-<instance part="SV5" gate="1" x="-106.68" y="119.38"/>
-<instance part="SV6" gate="1" x="-76.2" y="119.38" rot="MR0"/>
+<instance part="SV5" gate="1" x="-233.68" y="-2.54"/>
+<instance part="SV6" gate="1" x="-200.66" y="-2.54" rot="MR0"/>
 <instance part="SV7" gate="1" x="-106.68" y="-5.08"/>
 <instance part="SV8" gate="1" x="-114.3" y="-5.08" rot="MR0"/>
@@
 <instance part="SV12" gate="1" x="241.3" y="160.02" rot="MR0"/>
 <instance part="GND4" gate="1" x="-137.16" y="66.04"/>
-<instance part="P+13" gate="1" x="-86.36" y="127"/>
-<instance part="P-10" gate="1" x="-86.36" y="109.22"/>
-<instance part="GND31" gate="1" x="-96.52" y="109.22"/>
+<instance part="P+13" gate="1" x="-177.8" y="-2.54"/>
+<instance part="P-10" gate="1" x="-210.82" y="-12.7"/>
+<instance part="GND31" gate="1" x="-220.98" y="-12.7"/>
 <instance part="GND34" gate="1" x="223.52" y="152.4"/>
 <instance part="GND35" gate="1" x="269.24" y="152.4"/>
@@
 <instance part="IC3" gate="G$1" x="119.38" y="182.88"/>
 <instance part="C15" gate="G$1" x="203.2" y="142.24" rot="R270"/>
+<instance part="CENTER" gate="G$1" x="-187.96" y="-7.62" rot="R90"/>
+<instance part="GND14" gate="1" x="-187.96" y="2.54"/>
 </instances>
 <busses>
@@
 <pinref part="C20" gate="G$1" pin="2"/>
 <wire x1="-53.34" y1="134.62" x2="-53.34" y2="137.16" width="0.1524" layer="91"/>
-<pinref part="C19" gate="G$1" pin="2"/>
-<wire x1="-53.34" y1="139.7" x2="-53.34" y2="137.16" width="0.1524" layer="91"/>
 <junction x="-53.34" y="137.16"/>
 <pinref part="C9" gate="G$1" pin="+"/>
@@
 <pinref part="SV6" gate="1" pin="2"/>
 <pinref part="SV5" gate="1" pin="2"/>
-<wire x1="-83.82" y1="116.84" x2="-96.52" y2="116.84" width="0.1524" layer="91"/>
+<wire x1="-208.28" y1="-5.08" x2="-220.98" y2="-5.08" width="0.1524" layer="91"/>
 <pinref part="GND31" gate="1" pin="GND"/>
-<wire x1="-96.52" y1="116.84" x2="-99.06" y2="116.84" width="0.1524" layer="91"/>
-<wire x1="-96.52" y1="111.76" x2="-96.52" y2="116.84" width="0.1524" layer="91"/>
+<wire x1="-220.98" y1="-5.08" x2="-226.06" y2="-5.08" width="0.1524" layer="91"/>
+<wire x1="-220.98" y1="-10.16" x2="-220.98" y2="-5.08" width="0.1524" layer="91"/>
 <pinref part="SV5" gate="1" pin="3"/>
 <pinref part="SV6" gate="1" pin="3"/>
-<wire x1="-99.06" y1="119.38" x2="-96.52" y2="119.38" width="0.1524" layer="91"/>
-<wire x1="-96.52" y1="119.38" x2="-83.82" y2="119.38" width="0.1524" layer="91"/>
-<wire x1="-96.52" y1="116.84" x2="-96.52" y2="119.38" width="0.1524" layer="91"/>
-<junction x="-96.52" y="116.84"/>
-<junction x="-96.52" y="119.38"/>
+<wire x1="-226.06" y1="-2.54" x2="-220.98" y2="-2.54" width="0.1524" layer="91"/>
+<wire x1="-220.98" y1="-2.54" x2="-208.28" y2="-2.54" width="0.1524" layer="91"/>
+<wire x1="-220.98" y1="-5.08" x2="-220.98" y2="-2.54" width="0.1524" layer="91"/>
+<junction x="-220.98" y="-5.08"/>
+<junction x="-220.98" y="-2.54"/>
 </segment>
 <segment>
@@
 <junction x="-139.7" y="43.18"/>
 </segment>
+<segment>
+<pinref part="GND14" gate="1" pin="GND"/>
+<pinref part="C19" gate="G$1" pin="2"/>
+<wire x1="-187.96" y1="5.08" x2="-187.96" y2="7.62" width="0.1524" layer="91"/>
+</segment>
 </net>
 <net name="N$16" class="0">
@@
 <junction x="-25.4" y="149.86"/>
 <junction x="-33.02" y="149.86"/>
-<pinref part="C19" gate="G$1" pin="1"/>
-<wire x1="-53.34" y1="147.32" x2="-53.34" y2="149.86" width="0.1524" layer="91"/>
-<wire x1="-53.34" y1="149.86" x2="-43.18" y2="149.86" width="0.1524" layer="91"/>
-<junction x="-43.18" y="149.86"/>
 <pinref part="C10" gate="G$1" pin="+"/>
 </segment>
@@
 </segment>
 <segment>
-<pinref part="SV6" gate="1" pin="4"/>
-<pinref part="P+13" gate="1" pin="+12V"/>
-<wire x1="-83.82" y1="121.92" x2="-86.36" y2="121.92" width="0.1524" layer="91"/>
-<wire x1="-86.36" y1="121.92" x2="-86.36" y2="124.46" width="0.1524" layer="91"/>
-<pinref part="SV5" gate="1" pin="4"/>
-<wire x1="-99.06" y1="121.92" x2="-86.36" y2="121.92" width="0.1524" layer="91"/>
-<junction x="-86.36" y="121.92"/>
-</segment>
-<segment>
 <pinref part="P+7" gate="1" pin="+12V"/>
 <pinref part="IC2" gate="A" pin="V+"/>
@@
 </segment>
 <segment>
-<pinref part="R47" gate="G$1" pin="2"/>
-<wire x1="-149.86" y1="17.78" x2="-149.86" y2="15.24" width="0.1524" layer="91"/>
-<pinref part="P+9" gate="1" pin="+12V"/>
+<pinref part="CENTER" gate="G$1" pin="A"/>
+<wire x1="-180.34" y1="-7.62" x2="-177.8" y2="-7.62" width="0.1524" layer="91"/>
+<pinref part="P+13" gate="1" pin="+12V"/>
+<wire x1="-177.8" y1="-7.62" x2="-177.8" y2="-5.08" width="0.1524" layer="91"/>
 </segment>
 </net>
@@
 <pinref part="SV5" gate="1" pin="1"/>
 <pinref part="P-10" gate="1" pin="-12V"/>
-<wire x1="-99.06" y1="114.3" x2="-86.36" y2="114.3" width="0.1524" layer="91"/>
-<wire x1="-86.36" y1="114.3" x2="-86.36" y2="111.76" width="0.1524" layer="91"/>
+<wire x1="-226.06" y1="-7.62" x2="-210.82" y2="-7.62" width="0.1524" layer="91"/>
+<wire x1="-210.82" y1="-7.62" x2="-210.82" y2="-10.16" width="0.1524" layer="91"/>
 <pinref part="SV6" gate="1" pin="1"/>
-<wire x1="-83.82" y1="114.3" x2="-86.36" y2="114.3" width="0.1524" layer="91"/>
-<junction x="-86.36" y="114.3"/>
+<wire x1="-208.28" y1="-7.62" x2="-210.82" y2="-7.62" width="0.1524" layer="91"/>
+<junction x="-210.82" y="-7.62"/>
 </segment>
 <segment>
@@
 </segment>
 </net>
+<net name="N$40" class="0">
+<segment>
+<pinref part="R47" gate="G$1" pin="2"/>
+<wire x1="-149.86" y1="17.78" x2="-149.86" y2="15.24" width="0.1524" layer="91"/>
+<pinref part="CENTER" gate="G$1" pin="E"/>
+<wire x1="-195.58" y1="-7.62" x2="-195.58" y2="-2.54" width="0.1524" layer="91"/>
+<pinref part="CENTER" gate="G$1" pin="S"/>
+<wire x1="-195.58" y1="-2.54" x2="-187.96" y2="-2.54" width="0.1524" layer="91"/>
+<wire x1="-195.58" y1="-2.54" x2="-195.58" y2="7.62" width="0.1524" layer="91"/>
+<pinref part="SV6" gate="1" pin="4"/>
+<pinref part="SV5" gate="1" pin="4"/>
+<wire x1="-226.06" y1="0" x2="-213.36" y2="0" width="0.1524" layer="91"/>
+<wire x1="-213.36" y1="0" x2="-208.28" y2="0" width="0.1524" layer="91"/>
+<wire x1="-195.58" y1="7.62" x2="-213.36" y2="7.62" width="0.1524" layer="91"/>
+<wire x1="-213.36" y1="7.62" x2="-213.36" y2="0" width="0.1524" layer="91"/>
+<junction x="-195.58" y="-2.54"/>
+<junction x="-213.36" y="0"/>
+<wire x1="-149.86" y1="17.78" x2="-187.96" y2="17.78" width="0.1524" layer="91"/>
+<wire x1="-187.96" y1="17.78" x2="-213.36" y2="17.78" width="0.1524" layer="91"/>
+<wire x1="-213.36" y1="17.78" x2="-213.36" y2="7.62" width="0.1524" layer="91"/>
+<junction x="-213.36" y="7.62"/>
+<pinref part="C19" gate="G$1" pin="1"/>
+<wire x1="-187.96" y1="15.24" x2="-187.96" y2="17.78" width="0.1524" layer="91"/>
+<junction x="-187.96" y="17.78"/>
+</segment>
+</net>

Commit message: fixed the levels for the 3340 and vcf3
Parts:
- R18: value 10k -> 1k
- R19, R20: value 22k -> 47k
Changed lines of the file:
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@@
 <part name="R16" library="dan" deviceset="R-US_" device="0207/2V" value="10k"/>
 <part name="Q" library="dan" deviceset="US-EVU" device="F2J" value="10K"/>
-<part name="R18" library="dan" deviceset="R-US_" device="0207/2V" value="10k"/>
-<part name="R19" library="dan" deviceset="R-US_" device="0207/2V" value="22k"/>
-<part name="R20" library="dan" deviceset="R-US_" device="0207/2V" value="22k"/>
+<part name="R18" library="dan" deviceset="R-US_" device="0207/2V" value="1k"/>
+<part name="R19" library="dan" deviceset="R-US_" device="0207/2V" value="47k"/>
+<part name="R20" library="dan" deviceset="R-US_" device="0207/2V" value="47k"/>
 <part name="GND6" library="dan" deviceset="GND" device=""/>
 <part name="GAIN" library="dan" deviceset="US-EVU" device="F2J" value="10K"/>

Commit message: added tri and linear mod to vco, fixed serious errors with cvsource
Parts:
- R14, R15, R17, R29: value 47k -> 240k
- R26: value 22k -> 110k
Changed lines of the file:
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@@
 <part name="R12" library="dan" deviceset="R-US_" device="0207/2V" value="1k"/>
 <part name="R13" library="dan" deviceset="R-US_" device="0207/2V" value="1k"/>
-<part name="R14" library="dan" deviceset="R-US_" device="0207/2V" value="47k"/>
-<part name="R15" library="dan" deviceset="R-US_" device="0207/2V" value="47k"/>
+<part name="R14" library="dan" deviceset="R-US_" device="0207/2V" value="240k"/>
+<part name="R15" library="dan" deviceset="R-US_" device="0207/2V" value="240k"/>
 <part name="GND5" library="dan" deviceset="GND" device=""/>
 <part name="R16" library="dan" deviceset="R-US_" device="0207/2V" value="10k"/>
@@
 <part name="MIN" library="dan" deviceset="PJ301BM" device=""/>
 <part name="GND13" library="dan" deviceset="GND" device=""/>
-<part name="R29" library="dan" deviceset="R-US_" device="0207/2V" value="47k"/>
+<part name="R29" library="dan" deviceset="R-US_" device="0207/2V" value="240k"/>
 <part name="R30" library="dan" deviceset="R-US_" device="0207/2V" value="1k"/>
 <part name="R31" library="dan" deviceset="R-US_" device="0207/2V" value="1k"/>
-<part name="R17" library="dan" deviceset="R-US_" device="0207/2V" value="47k"/>
+<part name="R17" library="dan" deviceset="R-US_" device="0207/2V" value="240k"/>
 <part name="GND15" library="dan" deviceset="GND" device=""/>
 <part name="POWER" library="dan" deviceset="2516-" device=""/>
@@
 <part name="Q12" library="dan" deviceset="2N3904" device=""/>
 <part name="SCALE" library="dan" deviceset="TRIM_US-" device="S64W" value="500K"/>
-<part name="R26" library="dan" deviceset="R-US_" device="0207/2V" value="22k"/>
+<part name="R26" library="dan" deviceset="R-US_" device="0207/2V" value="110k"/>
 <part name="C9" library="dan" deviceset="CPOL-US" device="E2.5-6" value="4.7u"/>
 <part name="C10" library="dan" deviceset="CPOL-US" device="E2.5-6" value="4.7u"/>
