File: cvsource/cvsource.brd (EAGLE design)
At the start: 101.6 x 223.2 mm, 114 parts, among them IC1 OPA4130P, IC2 OPA2134P, IC3 78L05Z, P1 US-EVUF3J, P2 US-EVUF3J, P3 US-EVUF3J, P4 US-EVUF3J, X1 2516-

Commit message: ordered cvsource
Routing:
- net N$18: track 3.91 -> 3.19 mm, vias 1 -> 0
Other:
- board text added: "CV1"
- board text added: "CV2"
- board text added: "CV3"
- board text added: "CV4"
Changed lines of the file:
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@@
 <text x="24.13" y="153.67" size="1.778" layer="51" ratio="15" align="center">LFO</text>
 <text x="90.17" y="92.71" size="1.27" layer="21" font="vector" ratio="15" rot="R180">optional</text>
+<text x="24.13" y="129.54" size="1.778" layer="21" font="vector" ratio="15">CV1</text>
+<text x="39.37" y="129.54" size="1.778" layer="21" font="vector" ratio="15">CV2</text>
+<text x="54.61" y="129.54" size="1.778" layer="21" font="vector" ratio="15">CV3</text>
+<text x="69.85" y="129.54" size="1.778" layer="21" font="vector" ratio="15">CV4</text>
 </plain>
 <attributes>
@@
 <contactref element="MODE" pad="4"/>
 <contactref element="R44" pad="2"/>
-<wire x1="82.55" y1="184.15" x2="85.09" y2="184.15" width="0.6096" layer="16"/>
-<wire x1="85.09" y1="184.15" x2="85.1408" y2="185.5216" width="0.6096" layer="1"/>
-<via x="85.09" y="184.15" extent="1-16" drill="0.7"/>
+<wire x1="82.55" y1="184.15" x2="83.82" y2="184.15" width="0.6096" layer="16"/>
+<wire x1="83.82" y1="184.15" x2="85.09" y2="185.42" width="0.6096" layer="16"/>
+<wire x1="85.09" y1="185.42" x2="85.09" y2="185.4708" width="0.4064" layer="16"/>
+<wire x1="85.09" y1="185.4708" x2="85.1408" y2="185.5216" width="0.4064" layer="16"/>
 </signal>
 <signal name="N$12">
