File: 2045/2045.sch (EAGLE design)
At the start: 47 parts, among them IC1 OPA2134P, IC2 OPA2134P, X1 2516-

Commit message: upated the 2045 filter
Parts:
- added C13, C14: (no value), dan:CPOL-USE2.5-7
- added D4, D5, D6, D7: 1N4148DO35-7, dan:1N4148DO35-7
- added IN1POT, IN2POT: US-EVUF2J, dan:US-EVUF2J
- added R25, R51: 10, dan:R-US_0207/2V
- C5, C6, C7: device dan:CPOL-USE3.5-10 -> dan:CPOL-USE2.5-7
- R1, R10, R11, R12, R13, R14, R15, R2, R3, R4, R5, R6, R7, R8, R9: device dan:R-US_0309/12 -> dan:R-US_0204/7
Connections:
- new net N$35: IN.P$3, IN1POT.E
- new net N$36: IN2.P$3, IN2POT.E
- new net N$37: D6.C, D7.C, R51.2
- new net N$38: D4.A, D5.A, R25.2
- new net N$71: D7.A, X1-10.KL, X1-9.KL
- new net N$72: D4.C, X1-1.KL, X1-2.KL
- net +12V: now also C13.+, R51.1; no longer X1-10.KL, X1-9.KL
- net -12V: now also C14.-, R25.1; no longer X1-1.KL, X1-2.KL
- net GND: now also C13.-, C14.+, D5.C, D6.A, IN1POT.A, IN2POT.A
- net N$15: now also IN1POT.S; no longer IN.P$3
- net N$29: now also IN2POT.S; no longer IN2.P$3
Other:
- moved on the sheet: C10, C11, C12, C9, R8
